Commit message: Updating

File: box_car_description/robot/box_bot_body.xacro (robot description, xacro)
@@ -24,5 +24,5 @@
           </geometry> -->
           <geometry>
-            <mesh filename="/home/ros2_ws/src/box_car/box_car_description/meshes/box_car.dae" scale="1.0 1.0 1.0"/>
+            <mesh filename="package://box_car_description/meshes/box_car.dae" scale="1.0 1.0 1.0"/>
           </geometry>
         </visual>

File: box_car_description/robot/wheels.xacro (robot description, xacro)
@@ -21,5 +21,5 @@
             </geometry> -->
             <geometry>
-              <mesh filename="/home/ros2_ws/src/box_car/box_car_description/meshes/wheel.dae" scale="1.0 1.0 1.0"/>
+              <mesh filename="package://box_car_description/meshes/wheel.dae" scale="1.0 1.0 1.0"/>
             </geometry>
           </visual>
